Commit message: 清晰了urdf文件以及话题通信关系，解耦合了urdfws和moveit，将手部网格拷贝了

File: ROS/moveit_with_hand_ws/src/tianyi2_moveit_config/urdf/tianyi2.0_complete_with_hands.xacro (robot description, xacro)
@@ -2,5 +2,5 @@
 <robot name="tianyi2.0_complete" xmlns:xacro="http://wiki.ros.org/xacro">
   <xacro:arg name="flange_length" default="0.031" />
-  <xacro:include filename="$(find tianyi2_urdf)/urdf/tianyi2.0_URDF.urdf.xacro" />
+  <xacro:include filename="$(find tianyi2_moveit_config)/urdf/tianyi2.0_URDF.urdf.xacro" />
   <xacro:macro name="install_left_hand" params="parent:='left_tcp_link' xyz:='0 0 0' rpy:='0 0 0' flange_length:=0.031">
     <link name="L_base_link">
@@ -12,10 +12,10 @@
       <visual>
         <origin xyz="0 0 0" rpy="0 0 0" />
-        <geometry><mesh filename="package://tianyi2_urdf/meshes/L_base_link.STL" /></geometry>
-        <material name=""><color rgba="1 1 1 1" /></material>
-      </visual>
-      <collision>
-        <origin xyz="0 0 0" rpy="0 0 0" />
-        <geometry><mesh filename="package://tianyi2_urdf/meshes_convex/L_base_link.STL" /></geometry>
+        <geometry><mesh filename="package://tianyi2_moveit_config/meshes/L_base_link.STL" /></geometry>
+        <material name=""><color rgba="1 1 1 1" /></material>
+      </visual>
+      <collision>
+        <origin xyz="0 0 0" rpy="0 0 0" />
+        <geometry><mesh filename="package://tianyi2_moveit_config/meshes_convex/L_base_link.STL" /></geometry>
       </collision>
     </link>
@@ -29,10 +29,10 @@
       <visual>
         <origin xyz="0 0 0" rpy="0 0 0" />
-        <geometry><mesh filename="package://tianyi2_urdf/meshes/left_thumb_1.STL" /></geometry>
-        <material name=""><color rgba="1 1 1 1" /></material>
-      </visual>
-      <collision>
-        <origin xyz="0 0 0" rpy="0 0 0" />
-        <geometry><mesh filename="package://tianyi2_urdf/meshes_convex/left_thumb_1.STL" /></geometry>
+        <geometry><mesh filename="package://tianyi2_moveit_config/meshes/left_thumb_1.STL" /></geometry>
+        <material name=""><color rgba="1 1 1 1" /></material>
+      </visual>
+      <collision>
+        <origin xyz="0 0 0" rpy="0 0 0" />
+        <geometry><mesh filename="package://tianyi2_moveit_config/meshes_convex/left_thumb_1.STL" /></geometry>
       </collision>
     </link>
@@ -53,10 +53,10 @@
       <visual>
         <origin xyz="0 0 0" rpy="0 0 0" />
-        <geometry><mesh filename="package://tianyi2_urdf/meshes/left_thumb_2.STL" /></geometry>
-        <material name=""><color rgba="1 1 1 1" /></material>
-      </visual>
-      <collision>
-        <origin xyz="0 0 0" rpy="0 0 0" />
-        <geometry><mesh filename="package://tianyi2_urdf/meshes_convex/left_thumb_2.STL" /></geometry>
+        <geometry><mesh filename="package://tianyi2_moveit_config/meshes/left_thumb_2.STL" /></geometry>
+        <material name=""><color rgba="1 1 1 1" /></material>
+      </visual>
+      <collision>
+        <origin xyz="0 0 0" rpy="0 0 0" />
+        <geometry><mesh filename="package://tianyi2_moveit_config/meshes_convex/left_thumb_2.STL" /></geometry>
       </collision>
     </link>
@@ -77,10 +77,10 @@
       <visual>
         <origin xyz="0 0 0" rpy="0 0 0" />
-        <geometry><mesh filename="package://tianyi2_urdf/meshes/left_thumb_3.STL" /></geometry>
-        <material name=""><color rgba="1 1 1 1" /></material>
-      </visual>
-      <collision>
-        <origin xyz="0 0 0" rpy="0 0 0" />
-        <geometry><mesh filename="package://tianyi2_urdf/meshes_convex/left_thumb_3.STL" /></geometry>
+        <geometry><mesh filename="package://tianyi2_moveit_config/meshes/left_thumb_3.STL" /></geometry>
+        <material name=""><color rgba="1 1 1 1" /></material>
+      </visual>
+      <collision>
+        <origin xyz="0 0 0" rpy="0 0 0" />
+        <geometry><mesh filename="package://tianyi2_moveit_config/meshes_convex/left_thumb_3.STL" /></geometry>
       </collision>
     </link>
@@ -102,10 +102,10 @@
       <visual>
         <origin xyz="0 0 0" rpy="0 0 0" />
-        <geometry><mesh filename="package://tianyi2_urdf/meshes/left_thumb_4.STL" /></geometry>
-        <material name=""><color rgba="1 1 1 1" /></material>
-      </visual>
-      <collision>
-        <origin xyz="0 0 0" rpy="0 0 0" />
-        <geometry><mesh filename="package://tianyi2_urdf/meshes_convex/left_thumb_4.STL" /></geometry>
+        <geometry><mesh filename="package://tianyi2_moveit_config/meshes/left_thumb_4.STL" /></geometry>
+        <material name=""><color rgba="1 1 1 1" /></material>
+      </visual>
+      <collision>
+        <origin xyz="0 0 0" rpy="0 0 0" />
+        <geometry><mesh filename="package://tianyi2_moveit_config/meshes_convex/left_thumb_4.STL" /></geometry>
       </collision>
     </link>
@@ -127,10 +127,10 @@
       <visual>
         <origin xyz="0 0 0" rpy="0 0 0" />
-        <geometry><mesh filename="package://tianyi2_urdf/meshes/left_index_1.STL" /></geometry>
-        <material name=""><color rgba="1 1 1 1" /></material>
-      </visual>
-      <collision>
-        <origin xyz="0 0 0" rpy="0 0 0" />
-        <geometry><mesh filename="package://tianyi2_urdf/meshes_convex/left_index_1.STL" /></geometry>
+        <geometry><mesh filename="package://tianyi2_moveit_config/meshes/left_index_1.STL" /></geometry>
+        <material name=""><color rgba="1 1 1 1" /></material>
+      </visual>
+      <collision>
+        <origin xyz="0 0 0" rpy="0 0 0" />
+        <geometry><mesh filename="package://tianyi2_moveit_config/meshes_convex/left_index_1.STL" /></geometry>
       </collision>
     </link>
@@ -151,10 +151,10 @@
       <visual>
         <origin xyz="0 0 0" rpy="0 0 0" />
-        <geometry><mesh filename="package://tianyi2_urdf/meshes/left_index_2.STL" /></geometry>
-        <material name=""><color rgba="1 1 1 1" /></material>
-      </visual>
-      <collision>
-        <origin xyz="0 0 0" rpy="0 0 0" />
-        <geometry><mesh filename="package://tianyi2_urdf/meshes_convex/left_index_2.STL" /></geometry>
+        <geometry><mesh filename="package://tianyi2_moveit_config/meshes/left_index_2.STL" /></geometry>
+        <material name=""><color rgba="1 1 1 1" /></material>
+      </visual>
+      <collision>
+        <origin xyz="0 0 0" rpy="0 0 0" />
+        <geometry><mesh filename="package://tianyi2_moveit_config/meshes_convex/left_index_2.STL" /></geometry>
       </collision>
     </link>
@@ -176,10 +176,10 @@
       <visual>
         <origin xyz="0 0 0" rpy="0 0 0" />
-        <geometry><mesh filename="package://tianyi2_urdf/meshes/left_middle_1.STL" /></geometry>
-        <material name=""><color rgba="1 1 1 1" /></material>
-      </visual>
-      <collision>
-        <origin xyz="0 0 0" rpy="0 0 0" />
-        <geometry><mesh filename="package://tianyi2_urdf/meshes_convex/left_middle_1.STL" /></geometry>
+        <geometry><mesh filename="package://tianyi2_moveit_config/meshes/left_middle_1.STL" /></geometry>
+        <material name=""><color rgba="1 1 1 1" /></material>
+      </visual>
+      <collision>
+        <origin xyz="0 0 0" rpy="0 0 0" />
+        <geometry><mesh filename="package://tianyi2_moveit_config/meshes_convex/left_middle_1.STL" /></geometry>
       </collision>
     </link>
@@ -200,10 +200,10 @@
       <visual>
         <origin xyz="0 0 0" rpy="0 0 0" />
-        <geometry><mesh filename="package://tianyi2_urdf/meshes/left_middle_2.STL" /></geometry>
-        <material name=""><color rgba="1 1 1 1" /></material>
-      </visual>
-      <collision>
-        <origin xyz="0 0 0" rpy="0 0 0" />
-        <geometry><mesh filename="package://tianyi2_urdf/meshes_convex/left_middle_2.STL" /></geometry>
+        <geometry><mesh filename="package://tianyi2_moveit_config/meshes/left_middle_2.STL" /></geometry>
+        <material name=""><color rgba="1 1 1 1" /></material>
+      </visual>
+      <collision>
+        <origin xyz="0 0 0" rpy="0 0 0" />
+        <geometry><mesh filename="package://tianyi2_moveit_config/meshes_convex/left_middle_2.STL" /></geometry>
       </collision>
     </link>
@@ -225,10 +225,10 @@
       <visual>
         <origin xyz="0 0 0" rpy="0 0 0" />
-        <geometry><mesh filename="package://tianyi2_urdf/meshes/left_ring_1.STL" /></geometry>
-        <material name=""><color rgba="1 1 1 1" /></material>
-      </visual>
-      <collision>
-        <origin xyz="0 0 0" rpy="0 0 0" />
-        <geometry><mesh filename="package://tianyi2_urdf/meshes_convex/left_ring_1.STL" /></geometry>
+        <geometry><mesh filename="package://tianyi2_moveit_config/meshes/left_ring_1.STL" /></geometry>
+        <material name=""><color rgba="1 1 1 1" /></material>
+      </visual>
+      <collision>
+        <origin xyz="0 0 0" rpy="0 0 0" />
+        <geometry><mesh filename="package://tianyi2_moveit_config/meshes_convex/left_ring_1.STL" /></geometry>
       </collision>
     </link>
@@ -249,10 +249,10 @@
       <visual>
         <origin xyz="0 0 0" rpy="0 0 0" />
-        <geometry><mesh filename="package://tianyi2_urdf/meshes/left_ring_2.STL" /></geometry>
-        <material name=""><color rgba="1 1 1 1" /></material>
-      </visual>
-      <collision>
-        <origin xyz="0 0 0" rpy="0 0 0" />
-        <geometry><mesh filename="package://tianyi2_urdf/meshes_convex/left_ring_2.STL" /></geometry>
+        <geometry><mesh filename="package://tianyi2_moveit_config/meshes/left_ring_2.STL" /></geometry>
+        <material name=""><color rgba="1 1 1 1" /></material>
+      </visual>
+      <collision>
+        <origin xyz="0 0 0" rpy="0 0 0" />
+        <geometry><mesh filename="package://tianyi2_moveit_config/meshes_convex/left_ring_2.STL" /></geometry>
       </collision>
     </link>
@@ -274,10 +274,10 @@
       <visual>
         <origin xyz="0 0 0" rpy="0 0 0" />
-        <geometry><mesh filename="package://tianyi2_urdf/meshes/left_little_1.STL" /></geometry>
-        <material name=""><color rgba="1 1 1 1" /></material>
-      </visual>
-      <collision>
-        <origin xyz="0 0 0" rpy="0 0 0" />
-        <geometry><mesh filename="package://tianyi2_urdf/meshes_convex/left_little_1.STL" /></geometry>
+        <geometry><mesh filename="package://tianyi2_moveit_config/meshes/left_little_1.STL" /></geometry>
+        <material name=""><color rgba="1 1 1 1" /></material>
+      </visual>
+      <collision>
+        <origin xyz="0 0 0" rpy="0 0 0" />
+        <geometry><mesh filename="package://tianyi2_moveit_config/meshes_convex/left_little_1.STL" /></geometry>
       </collision>
     </link>
@@ -298,10 +298,10 @@
       <visual>
         <origin xyz="0 0 0" rpy="0 0 0" />
-        <geometry><mesh filename="package://tianyi2_urdf/meshes/left_little_2.STL" /></geometry>
-        <material name=""><color rgba="1 1 1 1" /></material>
-      </visual>
-      <collision>
-        <origin xyz="0 0 0" rpy="0 0 0" />
-        <geometry><mesh filename="package://tianyi2_urdf/meshes_convex/left_little_2.STL" /></geometry>
+        <geometry><mesh filename="package://tianyi2_moveit_config/meshes/left_little_2.STL" /></geometry>
+        <material name=""><color rgba="1 1 1 1" /></material>
+      </visual>
+      <collision>
+        <origin xyz="0 0 0" rpy="0 0 0" />
+        <geometry><mesh filename="package://tianyi2_moveit_config/meshes_convex/left_little_2.STL" /></geometry>
       </collision>
     </link>
@@ -359,10 +359,10 @@
       <visual>
         <origin xyz="0 0 0" rpy="0 0 0" />
-        <geometry><mesh filename="package://tianyi2_urdf/meshes/R_base_link.STL" /></geometry>
-        <material name=""><color rgba="1 1 1 1" /></material>
-      </visual>
-      <collision>
-        <origin xyz="0 0 0" rpy="0 0 0" />
-        <geometry><mesh filename="package://tianyi2_urdf/meshes_convex/R_base_link.STL" /></geometry>
+        <geometry><mesh filename="package://tianyi2_moveit_config/meshes/R_base_link.STL" /></geometry>
+        <material name=""><color rgba="1 1 1 1" /></material>
+      </visual>
+      <collision>
+        <origin xyz="0 0 0" rpy="0 0 0" />
+        <geometry><mesh filename="package://tianyi2_moveit_config/meshes_convex/R_base_link.STL" /></geometry>
       </collision>
     </link>
@@ -376,10 +376,10 @@
       <visual>
         <origin xyz="0 0 0" rpy="0 0 0" />
-        <geometry><mesh filename="package://tianyi2_urdf/meshes/right_thumb_1.STL" /></geometry>
-        <material name=""><color rgba="1 1 1 1" /></material>
-      </visual>
-      <collision>
-        <origin xyz="0 0 0" rpy="0 0 0" />
-        <geometry><mesh filename="package://tianyi2_urdf/meshes_convex/right_thumb_1.STL" /></geometry>
+        <geometry><mesh filename="package://tianyi2_moveit_config/meshes/right_thumb_1.STL" /></geometry>
+        <material name=""><color rgba="1 1 1 1" /></material>
+      </visual>
+      <collision>
+        <origin xyz="0 0 0" rpy="0 0 0" />
+        <geometry><mesh filename="package://tianyi2_moveit_config/meshes_convex/right_thumb_1.STL" /></geometry>
       </collision>
     </link>
@@ -400,10 +400,10 @@
       <visual>
         <origin xyz="0 0 0" rpy="0 0 0" />
-        <geometry><mesh filename="package://tianyi2_urdf/meshes/right_thumb_2.STL" /></geometry>
-        <material name=""><color rgba="1 1 1 1" /></material>
-      </visual>
-      <collision>
-        <origin xyz="0 0 0" rpy="0 0 0" />
-        <geometry><mesh filename="package://tianyi2_urdf/meshes_convex/right_thumb_2.STL" /></geometry>
+        <geometry><mesh filename="package://tianyi2_moveit_config/meshes/right_thumb_2.STL" /></geometry>
+        <material name=""><color rgba="1 1 1 1" /></material>
+      </visual>
+      <collision>
+        <origin xyz="0 0 0" rpy="0 0 0" />
+        <geometry><mesh filename="package://tianyi2_moveit_config/meshes_convex/right_thumb_2.STL" /></geometry>
       </collision>
     </link>
@@ -423,10 +423,10 @@
       <visual>
         <origin xyz="0 0 0" rpy="0 0 0" />
-        <geometry><mesh filename="package://tianyi2_urdf/meshes/right_thumb_3.STL" /></geometry>
-        <material name=""><color rgba="1 1 1 1" /></material>
-      </visual>
-      <collision>
-        <origin xyz="0 0 0" rpy="0 0 0" />
-        <geometry><mesh filename="package://tianyi2_urdf/meshes_convex/right_thumb_3.STL" /></geometry>
+        <geometry><mesh filename="package://tianyi2_moveit_config/meshes/right_thumb_3.STL" /></geometry>
+        <material name=""><color rgba="1 1 1 1" /></material>
+      </visual>
+      <collision>
+        <origin xyz="0 0 0" rpy="0 0 0" />
+        <geometry><mesh filename="package://tianyi2_moveit_config/meshes_convex/right_thumb_3.STL" /></geometry>
       </collision>
     </link>
@@ -448,10 +448,10 @@
       <visual>
         <origin xyz="0 0 0" rpy="0 0 0" />
-        <geometry><mesh filename="package://tianyi2_urdf/meshes/right_thumb_4.STL" /></geometry>
-        <material name=""><color rgba="1 1 1 1" /></material>
-      </visual>
-      <collision>
-        <origin xyz="0 0 0" rpy="0 0 0" />
-        <geometry><mesh filename="package://tianyi2_urdf/meshes_convex/right_thumb_4.STL" /></geometry>
+        <geometry><mesh filename="package://tianyi2_moveit_config/meshes/right_thumb_4.STL" /></geometry>
+        <material name=""><color rgba="1 1 1 1" /></material>
+      </visual>
+      <collision>
+        <origin xyz="0 0 0" rpy="0 0 0" />
+        <geometry><mesh filename="package://tianyi2_moveit_config/meshes_convex/right_thumb_4.STL" /></geometry>
       </collision>
     </link>
@@ -473,10 +473,10 @@
       <visual>
         <origin xyz="0 0 0" rpy="0 0 0" />
-        <geometry><mesh filename="package://tianyi2_urdf/meshes/right_index_1.STL" /></geometry>
-        <material name=""><color rgba="1 1 1 1" /></material>
-      </visual>
-      <collision>
-        <origin xyz="0 0 0" rpy="0 0 0" />
-        <geometry><mesh filename="package://tianyi2_urdf/meshes_convex/right_index_1.STL" /></geometry>
+        <geometry><mesh filename="package://tianyi2_moveit_config/meshes/right_index_1.STL" /></geometry>
+        <material name=""><color rgba="1 1 1 1" /></material>
+      </visual>
+      <collision>
+        <origin xyz="0 0 0" rpy="0 0 0" />
+        <geometry><mesh filename="package://tianyi2_moveit_config/meshes_convex/right_index_1.STL" /></geometry>
       </collision>
     </link>
@@ -497,10 +497,10 @@
       <visual>
         <origin xyz="0 0 0" rpy="0 0 0" />
-        <geometry><mesh filename="package://tianyi2_urdf/meshes/right_index_2.STL" /></geometry>
-        <material name=""><color rgba="1 1 1 1" /></material>
-      </visual>
-      <collision>
-        <origin xyz="0 0 0" rpy="0 0 0" />
-        <geometry><mesh filename="package://tianyi2_urdf/meshes_convex/right_index_2.STL" /></geometry>
+        <geometry><mesh filename="package://tianyi2_moveit_config/meshes/right_index_2.STL" /></geometry>
+        <material name=""><color rgba="1 1 1 1" /></material>
+      </visual>
+      <collision>
+        <origin xyz="0 0 0" rpy="0 0 0" />
+        <geometry><mesh filename="package://tianyi2_moveit_config/meshes_convex/right_index_2.STL" /></geometry>
       </collision>
     </link>
@@ -522,10 +522,10 @@
       <visual>
         <origin xyz="0 0 0" rpy="0 0 0" />
-        <geometry><mesh filename="package://tianyi2_urdf/meshes/right_middle_1.STL" /></geometry>
-        <material name=""><color rgba="1 1 1 1" /></material>
-      </visual>
-      <collision>
-        <origin xyz="0 0 0" rpy="0 0 0" />
-        <geometry><mesh filename="package://tianyi2_urdf/meshes_convex/right_middle_1.STL" /></geometry>
+        <geometry><mesh filename="package://tianyi2_moveit_config/meshes/right_middle_1.STL" /></geometry>
+        <material name=""><color rgba="1 1 1 1" /></material>
+      </visual>
+      <collision>
+        <origin xyz="0 0 0" rpy="0 0 0" />
+        <geometry><mesh filename="package://tianyi2_moveit_config/meshes_convex/right_middle_1.STL" /></geometry>
       </collision>
     </link>
@@ -546,10 +546,10 @@
       <visual>
         <origin xyz="0 0 0" rpy="0 0 0" />
-        <geometry><mesh filename="package://tianyi2_urdf/meshes/right_middle_2.STL" /></geometry>
-        <material name=""><color rgba="1 1 1 1" /></material>
-      </visual>
-      <collision>
-        <origin xyz="0 0 0" rpy="0 0 0" />
-        <geometry><mesh filename="package://tianyi2_urdf/meshes_convex/right_middle_2.STL" /></geometry>
+        <geometry><mesh filename="package://tianyi2_moveit_config/meshes/right_middle_2.STL" /></geometry>
+        <material name=""><color rgba="1 1 1 1" /></material>
+      </visual>
+      <collision>
+        <origin xyz="0 0 0" rpy="0 0 0" />
+        <geometry><mesh filename="package://tianyi2_moveit_config/meshes_convex/right_middle_2.STL" /></geometry>
       </collision>
     </link>
@@ -571,10 +571,10 @@
       <visual>
         <origin xyz="0 0 0" rpy="0 0 0" />
-        <geometry><mesh filename="package://tianyi2_urdf/meshes/right_ring_1.STL" /></geometry>
-        <material name=""><color rgba="1 1 1 1" /></material>
-      </visual>
-      <collision>
-        <origin xyz="0 0 0" rpy="0 0 0" />
-        <geometry><mesh filename="package://tianyi2_urdf/meshes_convex/right_ring_1.STL" /></geometry>
+        <geometry><mesh filename="package://tianyi2_moveit_config/meshes/right_ring_1.STL" /></geometry>
+        <material name=""><color rgba="1 1 1 1" /></material>
+      </visual>
+      <collision>
+        <origin xyz="0 0 0" rpy="0 0 0" />
+        <geometry><mesh filename="package://tianyi2_moveit_config/meshes_convex/right_ring_1.STL" /></geometry>
       </collision>
     </link>
@@ -595,10 +595,10 @@
       <visual>
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